File: KiCAD/pixdel6.sch (KiCad schematic (older format))
At the start: 13 parts, among them P1 ICSP, P2 chain_input, P3 chain_output, U1 PIC12F1572

Commit message: modification schématique
Parts:
- removed P1: ICSP, symbol CONN_M6
- removed R2: 470, symbol R
- removed R3: 180, symbol R
- removed R4: 150, symbol R
- removed R5: 67, symbol R
Connections:
- net PGCLK is gone; now on net blue: U1.6 (RA1)
- net PGDAT is gone; now on net green: U1.7 (RA0)
- net Vpp is gone; now on an unnamed net: U1.4 (RA3)
- net red: now also D1.1 (RED_ANODE)
- net blue: now reaches D1.4 (GREEN_ANODE)
- net green: now reaches D1.3 (BLUE_ANODE)
- no-connect marks 1 -> 0
Changed lines of the file:
@@
 LIBS:contrib
 LIBS:valves
-LIBS:librairie-personnelle
+LIBS:pixdel6-cache
 EELAYER 25 0
 EELAYER END
@@
 Wire Wire Line
 	6500 3200 6700 3200
-$Comp
-L R R4
-U 1 1 57E14FBE
-P 6900 3650
-F 0 "R4" V 6980 3650 50  0000 C CNN
-F 1 "150" V 6900 3650 50  0000 C CNN
-F 2 "" V 6830 3650 50  0000 C CNN
-F 3 "" H 6900 3650 50  0000 C CNN
-	1    6900 3650
-	1    0    0    -1
-$EndComp
-$Comp
-L R R3
-U 1 1 57E14FEC
-P 6700 3650
-F 0 "R3" V 6780 3650 50  0000 C CNN
-F 1 "180" V 6700 3650 50  0000 C CNN
-F 2 "" V 6630 3650 50  0000 C CNN
-F 3 "" H 6700 3650 50  0000 C CNN
-	1    6700 3650
-	1    0    0    -1
-$EndComp
-$Comp
-L R R5
-U 1 1 57E15054
-P 7100 3650
-F 0 "R5" V 7180 3650 50  0000 C CNN
-F 1 "67" V 7100 3650 50  0000 C CNN
-F 2 "" V 7030 3650 50  0000 C CNN
-F 3 "" H 7100 3650 50  0000 C CNN
-	1    7100 3650
-	1    0    0    -1
-$EndComp
 Wire Wire Line
 	6500 3500 6700 3500
 Wire Wire Line
-	6900 3500 6900 3400
+	6900 3400 6900 3950
 Wire Wire Line
 	6900 3400 6500 3400
@@
 	6500 3300 7100 3300
 Wire Wire Line
-	7100 3300 7100 3500
-Wire Wire Line
-	6700 3800 6700 3950
-Wire Wire Line
-	6900 3800 6900 3950
-Wire Wire Line
-	7100 3800 7100 3950
+	7100 3300 7100 3950
+Wire Wire Line
+	6700 3500 6700 3950
 $Comp
 L GND #PWR6
@@
 $EndComp
 $Comp
-L R R2
-U 1 1 57E152A8
-P 5300 3500
-F 0 "R2" V 5380 3500 50  0000 C CNN
-F 1 "470" V 5300 3500 50  0000 C CNN
-F 2 "" V 5230 3500 50  0000 C CNN
-F 3 "" H 5300 3500 50  0000 C CNN
-	1    5300 3500
-	0    1    1    0
-$EndComp
-$Comp
 L R R1
 U 1 1 57E152E8
@@
 	4950 3500 4950 3700
 Wire Wire Line
-	5150 3500 4950 3500
-Wire Wire Line
-	5450 3500 5650 3500
+	4950 3500 5650 3500
 Wire Wire Line
 	4950 3200 4950 2950
@@
 Text Label 6700 3500 0    60   ~ 0
 red
-Text Label 6850 3400 0    60   ~ 0
+Text Label 7100 3300 0    60   ~ 0
 green
-Text Label 7100 3300 0    60   ~ 0
+Text Label 6900 3400 0    60   ~ 0
 blue
-$Comp
-L CONN_M6 P1
-U 1 1 57E1653B
-P 3950 4500
-F 0 "P1" H 3975 4100 50  0000 C CNN
-F 1 "ICSP" H 3975 4800 50  0000 C CNN
-F 2 "" H 3950 4500 60  0001 C CNN
-F 3 "" H 3950 4500 60  0001 C CNN
-	1    3950 4500
-	1    0    0    -1
-$EndComp
-Text Label 4200 4300 0    50   ~ 0
-Vpp
-Text Label 4200 4400 0    50   ~ 0
-Vdd
-Text Label 4200 4500 0    50   ~ 0
-Vss
-Text Label 4200 4700 0    50   ~ 0
-PGCLK
-Text Label 4200 4600 0    50   ~ 0
-PGDAT
-NoConn ~ 4200 4800
-Text Label 5650 3500 2    50   ~ 0
-Vpp
-Text Label 6500 3300 0    50   ~ 0
-PGDAT
-Text Label 6500 3400 0    50   ~ 0
-PGCLK
 Text Label 5650 3200 2    50   ~ 0
 Vdd
